File: HW/Chorus_CH32.kicad_sch (KiCad schematic)
At the start: 19 parts, among them J1 DC_Jack, U1 CH32V003JxMx, U2 TSR_1-2450, U3 TL072

Commit message: pre-schematic + pre-layout
Parts:
- removed U2: TSR_1-2450, Converter_DCDC:Converter_DCDC_TRACO_TSR-1_THT, symbol Regulator_Switching:TSR_1-2450
- removed U3: TL072, symbol Amplifier_Operational:TL072
- added C10, C11, C9: 100n, Capacitor_SMD:C_0603_1608Metric, symbol Device:C
- added C7, C8: 22u, Capacitor_SMD:C_1210_3225Metric, symbol Device:C
- added D2: CTL1, LED_SMD:LED_0603_1608Metric, symbol Device:LED
- added D3: LED, LED_SMD:LED_0603_1608Metric, symbol Device:LED
- added D4: 1N5819WS, Diode_SMD:D_SOD-323, symbol Device:D
- added J2: Prog_Head, Connector_PinSocket_1.27mm:PinSocket_1x03_P1.27mm_Vertical, symbol Connector:Conn_01x03_Socket
- added J3: Footswitch, Connector_JST:JST_PH_B2B-PH-K_1x02_P2.00mm_Vertical, symbol Connector:Conn_01x02_Pin
- added K1: G6KU-2, Relay_SMD:Relay_DPDT_Omron_G6K-2F-Y, symbol Relay:G6KU-2
- added U2: TPS82130, Package_LGA:Texas_SIL0008D_MicroSiP-8-1EP_2.8x3mm_P0.65mm_EP1.1x1.9mm_ThermalVias, symbol Regulator_Switching:TPS82130
- added U3, U5: TL074, Package_SO:SOIC-14_3.9x8.7mm_P1.27mm, symbol Amplifier_Operational:TL074
- added U4: 74LVC2G00, Package_SO:VSSOP-8_2.3x2mm_P0.5mm, symbol 74xGxx:74LVC2G00
- Audio1, Audio2: footprint AREA_lib_composant:AUDIO-TH_PJ-603A_1 -> easyeda2kicad:AUDIO-TH_PJ-603A
- C3: value 100n -> 430p
- R1, R4: value 10M -> 330; footprint (none) -> Resistor_SMD:R_0603_1608Metric
- R2: value 39K -> TBD; footprint (none) -> Resistor_SMD:R_0603_1608Metric
- R3: value 15K -> TBD; footprint (none) -> Resistor_SMD:R_0603_1608Metric
- R5: value 1k -> 523K; footprint (none) -> Resistor_SMD:R_0603_1608Metric
- R6: value 10k -> 100K; footprint (none) -> Resistor_SMD:R_0603_1608Metric
- U1: footprint Package_SO:SOP-8_3.9x4.9mm_P1.27mm -> Package_SO:SOP-16_3.9x9.9mm_P1.27mm; symbol MCU_WCH_CH32V0:CH32V003JxMx -> MCU_WCH_CH32V0:CH32V003AxMx
Connections:
- net +5V: now also R5.2, U1.15 (VDD), C10.1, C8.1, C9.1, J2.1 (Pin_1), J3.1 (Pin_1), U2.4 (VOUT), U2.5 (VOUT), U4.8 (VCC); no longer U1.4 (VDD)
- net +9V: now also C11.1, C7.1, U2.1 (EN), U2.2 (VIN), U3.4 (V+), U5.4 (V+)
- net ADC_IN: no longer R5.2, R6.1, U1.7 (PC4)
- net GND: now also C3.1, R6.1, U1.14 (VSS), C10.2, C11.2, C7.2, C8.2, C9.2, D2.1 (K), D3.1 (K), J2.3 (Pin_3), U2.3 (GND), U2.9 (GND), U3.11 (V-), U4.4 (GND), U5.11 (V-); no longer R1.2, R6.2, U1.2 (VSS)
- net IN: now also K1.3; no longer C3.1, R1.1
- net OUT: now also K1.6; no longer U1.5 (PC1)
- net at R5.1: now also R6.2, U2.6 (FB)
- net at R4.2: now also U1.10 (PD6); no longer C3.2
- net PWM_OUT_1: now reaches U1.1 (PC1)
- net SWITCH_OUT: now reaches U1.8 (PD4)
- net SWITCH_OUT: now also J3.2 (Pin_2)
- net +2V5 renamed TBD
- net TBD: no longer R4.1
- new net: D3.2 (A), R4.1
- new net: C3.2, U2.8 (SS/TR)
- new net: U1.13 (PA2), U4.5, U4.6
- new net: U1.12 (PA1), U4.1, U4.2
- new net: K1.2, K1.7
- new net: R1.1, U1.9 (PD5)
- new net: D2.2 (A), R1.2
- new net IN_FX: K1.4
- new net OUT_FX: K1.5
- new net PWM_OUT_2: U1.2 (PC2)
- new net RELAY_+: D4.1 (K), K1.1, U4.7
- new net RELAY_-: D4.2 (A), K1.8, U4.3
- new net SWDIO: J2.2 (Pin_2), U1.7 (PD1)
- no-connect marks 1 -> 2
Other:
- note removed: "Only for breadboard test"
- moved on the sheet: Audio1, Audio2, C4, C5
